Commit message: Update Spot MoveIt configuration files

File: spot-ros2_ws/src/spot_moveit_config/config/spot.ros2_control.xacro (robot description, xacro)
@@ -8,4 +8,11 @@
                 <plugin>mock_components/GenericSystem</plugin>
             </hardware>
+            <joint name="arm_sh0">
+                <command_interface name="position"/>
+                <state_interface name="position">
+                  <param name="initial_value">${initial_positions['arm_sh0']}</param>
+                </state_interface>
+                <state_interface name="velocity"/>
+            </joint>
             <joint name="arm_sh1">
                 <command_interface name="position"/>
